File: hw/sch_pcb/TFPROBE01.kicad_sch (KiCad schematic)
At the start: 8 parts, among them J1 HEADER_1x03, M3 HOLE, M4 HOLE, U1 AH3572, U2 VCNT2020

Commit message: Improve documentation quality.
Other:
- note added: "Hall effect omnipolar magnetic switch"
- note removed: "HALL EFFECT OMNIPOLAR SWITCH"
Changed lines of the file:
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@@
 		)
 	)
-	(text "HALL EFFECT OMNIPOLAR SWITCH"
+	(text "Hall effect omnipolar magnetic switch"
 		(exclude_from_sim no)
-		(at 107.95 48.26 0)
+		(at 134.62 54.61 0)
 		(effects
 			(font
@@
 	(text "Reflective Optical Sensor"
 		(exclude_from_sim no)
-		(at 106.68 95.25 0)
+		(at 124.46 96.52 0)
 		(effects
 			(font
